File: acmp_test_fixture/acmp_test_fixture.sch (KiCad schematic (older format))
At the start: 11 parts, among them J1 Conn_Coaxial, J2 Conn_Coaxial, Y1 AXS-3225-04-02

Commit message: initial pcb design for the test fixture
Parts:
- C1, C2: value C -> 33n
- R1, R6: value 159R -> 158R
- R2, R5: value 66R2 -> 66R5
Other:
- note added: "50 Ohm to VNA"
- note added: "Crystal sees 25 Ohm\nCL=19 pF"
- note removed: "50Ohm to VNA"
- note removed: "crystal sees 25Ohm"
Changed lines of the file:
@@
 P 7600 3950
 F 0 "R6" H 7670 3996 50  0000 L CNN
-F 1 "159R" H 7670 3905 50  0000 L CNN
+F 1 "158R" H 7670 3905 50  0000 L CNN
 F 2 "Resistor_SMD:R_0603_1608Metric" V 7530 3950 50  0001 C CNN
 F 3 "~" H 7600 3950 50  0001 C CNN
@@
 P 7350 3500
 F 0 "R5" V 7143 3500 50  0000 C CNN
-F 1 "66R2" V 7234 3500 50  0000 C CNN
+F 1 "66R5" V 7234 3500 50  0000 C CNN
 F 2 "Resistor_SMD:R_0603_1608Metric" V 7280 3500 50  0001 C CNN
 F 3 "~" H 7350 3500 50  0001 C CNN
@@
 P 4700 3950
 F 0 "R1" H 4770 3996 50  0000 L CNN
-F 1 "159R" H 4770 3905 50  0000 L CNN
+F 1 "158R" H 4770 3905 50  0000 L CNN
 F 2 "Resistor_SMD:R_0603_1608Metric" V 4630 3950 50  0001 C CNN
 F 3 "~" H 4700 3950 50  0001 C CNN
@@
 P 4950 3500
 F 0 "R2" V 4743 3500 50  0000 C CNN
-F 1 "66R2" V 4834 3500 50  0000 C CNN
+F 1 "66R5" V 4834 3500 50  0000 C CNN
 F 2 "Resistor_SMD:R_0603_1608Metric" V 4880 3500 50  0001 C CNN
 F 3 "~" H 4950 3500 50  0001 C CNN
@@
 P 5700 3950
 F 0 "C1" H 5815 3996 50  0000 L CNN
-F 1 "C" H 5815 3905 50  0000 L CNN
+F 1 "33n" H 5815 3905 50  0000 L CNN
 F 2 "Capacitor_SMD:C_0603_1608Metric" H 5738 3800 50  0001 C CNN
 F 3 "~" H 5700 3950 50  0001 C CNN
@@
 P 6600 3950
 F 0 "C2" H 6715 3996 50  0000 L CNN
-F 1 "C" H 6715 3905 50  0000 L CNN
+F 1 "33n" H 6715 3905 50  0000 L CNN
 F 2 "Capacitor_SMD:C_0603_1608Metric" H 6638 3800 50  0001 C CNN
 F 3 "~" H 6600 3950 50  0001 C CNN
@@
 Wire Wire Line
 	6150 4400 6600 4400
-Text Notes 6250 3250 0    50   ~ 0
-crystal sees 25Ohm
+Text Notes 5800 2900 0    50   ~ 0
+Crystal sees 25 Ohm\nCL=19 pF
 Text Notes 3500 3550 0    50   ~ 0
-50Ohm to VNA
-Text Notes 6000 3800 0    50   ~ 0
+50 Ohm to VNA
+Text Notes 5300 3500 0    50   ~ 0
 12.5Ohm
 Connection ~ 6150 4400
