File: acmp_test_fixture/AXS-3225-04-02-variant/acmp_test_fixture.kicad_pcb (KiCad board)
At the start: 2 copper layers, 38.1 x 33 mm, 15 parts, among them J1 Conn_Coaxial, J2 Conn_Coaxial, Y1 AXS-3225-04-02

Commit message: added variant of test fixture
Changed lines of the file:
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@@
-(kicad_pcb (version 20171130) (host pcbnew "(5.1.4)-1")
+(kicad_pcb (version 20171130) (host pcbnew "(5.1.5)-3")
   (general
     (thickness 1.6)
-    (drawings 9)
+    (drawings 13)
     (tracks 6)
     (zones 0)
@@
   (page A4)
   (layers
-    (0 F.Cu signal)
-    (31 B.Cu signal)
+    (0 F.Cu signal hide)
+    (31 B.Cu signal hide)
     (32 B.Adhes user)
     (33 F.Adhes user)
@@
     (tags "mounting hole 3.2mm no annular m3")
     (attr virtual)
-    (fp_text reference REF** (at 0 -4.2) (layer F.SilkS)
+    (fp_text reference REF** (at 0 -4.2) (layer F.SilkS) hide
       (effects (font (size 1 1) (thickness 0.15)))
     )
@@
     (tags "mounting hole 3.2mm no annular m3")
     (attr virtual)
-    (fp_text reference REF** (at 0 -4.2) (layer F.SilkS)
+    (fp_text reference REF** (at 0 -4.2) (layer F.SilkS) hide
       (effects (font (size 1 1) (thickness 0.15)))
     )
@@
     (tags "mounting hole 3.2mm no annular m3")
     (attr virtual)
-    (fp_text reference REF** (at 0 -4.2) (layer F.SilkS)
+    (fp_text reference REF** (at 0 -4.2) (layer F.SilkS) hide
       (effects (font (size 1 1) (thickness 0.15)))
     )
@@
     (tags "mounting hole 3.2mm no annular m3")
     (attr virtual)
-    (fp_text reference REF** (at 0 -4.2) (layer F.SilkS)
+    (fp_text reference REF** (at 0 -4.2) (layer F.SilkS) hide
       (effects (font (size 1 1) (thickness 0.15)))
     )
@@
     (tags capacitor)
     (attr smd)
-    (fp_text reference C2 (at -0.0255 0 90) (layer F.SilkS)
+    (fp_text reference C2 (at 2.8955 0 90) (layer F.SilkS)
       (effects (font (size 1 1) (thickness 0.15)))
     )
@@
   (module abracon:AXS-3225-04-02 (layer F.Cu)
     (at 152.4 127 90)
-    (fp_text reference Y1 (at -8.255 0 180) (layer F.SilkS)
-      (effects (font (size 1 1) (thickness 0.15)))
-    )
-    (fp_text value AXS-3225-04-02 (at 0 -2.25 90) (layer F.Fab)
+    (fp_text reference Y1 (at 8.128 0 180) (layer F.SilkS)
+      (effects (font (size 1 1) (thickness 0.15)))
+    )
+    (fp_text value AXS-3225-04-02 (at 11.43 0 180) (layer F.SilkS)
       (effects (font (size 1 1) (thickness 0.15)))
     )
@@
       (net 1 "Net-(C1-Pad1)"))
   )
+  (gr_line (start 149.352 119.888) (end 149.352 134.112) (layer F.SilkS) (width 0.12))
+  (gr_line (start 155.448 119.888) (end 149.352 119.888) (layer F.SilkS) (width 0.12))
+  (gr_line (start 155.448 134.112) (end 155.448 119.888) (layer F.SilkS) (width 0.12))
+  (gr_line (start 149.352 134.112) (end 155.448 134.112) (layer F.SilkS) (width 0.12))
   (gr_line (start 133.35 114.3) (end 133.35 139.7) (layer Edge.Cuts) (width 0.15))
   (gr_line (start 167.64 110.49) (end 137.16 110.49) (layer Edge.Cuts) (width 0.15))
